File: sidekick.kicad_pcb (KiCad board)
At the start: 2 copper layers, 0 parts

Commit message: Add schematic and placeholder pcb
Parts:
- added BZ1: Buzzer, Buzzer_Beeper:Buzzer_12x9.5RM7.6, F.Cu at (191.9, 67.5)
- added R1: R, Resistor_THT:R_Axial_DIN0207_L6.3mm_D2.5mm_P7.62mm_Horizontal, F.Cu at (153.5, 96.5)
- added SW1: SW_PUSH_6mm_H5mm, Button_Switch_THT:SW_PUSH_6mm_H5mm, F.Cu at (128.5, 75.0)
- added SW2: SW_PUSH_6mm_H5mm, Button_Switch_THT:SW_PUSH_6mm_H5mm, F.Cu at (111.2, 85.8)
- added U1: ~, PCBCUPID-GLYPHC3-Footprint:GlyphC3, F.Cu at (69.8, 57.5)
- added U2: module_mpu6050, usini_sensors:module_mpu6050, F.Cu at (177.5, 94.0)
- added U3: DM-OLED096-636, DM-OLED096-636:MODULE_DM-OLED096-636, F.Cu at (175.2, 57.8)
