File: sidekick.kicad_pcb (KiCad board)
At the start: 2 copper layers, 7 parts, among them SW1 SW_PUSH_6mm_H5mm, SW2 SW_PUSH_6mm_H5mm, U2 module_mpu6050, U3 DM-OLED096-636

Commit message: Update to v0.2.5
Parts:
- added ?: , , F.Cu at (175.0, 121.0)
- added U3: DM-OLED096-636, DM-OLED096-636:MODULE_DM-OLED096-636, F.Cu at (111.5, 117.0)
- moved U1 104.5 mm to (155.7, 116.9)
- moved U3 83.7 mm to (116.0, 117.0), turned to -90 degrees
- moved BZ1 74.0 mm to (136.5, 116.5)
- moved SW1 55.2 mm to (162.8, 118.2)
- moved SW2 52.7 mm to (152.8, 118.2)
- moved R1 31.0 mm to (175.0, 118.8), turned to 90 degrees
- moved U2 30.1 mm to (152.0, 109.9)
Connections:
- SW1 pad 2: Net-(U1-D1) -> Net-(U1-D0)
- SW2 pad 2: Net-(U1-D0) -> Net-(U1-D1)
Routing:
- net Net-(U1-SDA): track 0.00 -> 75.5 mm
- net Net-(BZ1--): track 0.00 -> 70.5 mm
- net Net-(U2-VCC): track 0.00 -> 62.0 mm
- net Net-(U1-SCL): track 0.00 -> 58.1 mm
- net Net-(U1-D3): track 0.00 -> 40.8 mm
- net Net-(U1-D0): track 0.00 -> 15.8 mm
- net Net-(BZ1-+): track 0.00 -> 12.9 mm
- net Net-(U1-D1): track 0.00 -> 11.8 mm
- net Net-(U1-A2): track 0.00 -> 9.12 mm
Other:
- board outline added: 64.5 x 26.5 mm
- board text added: "GND"
- board text added: "SCL"
- board text added: "SDA"
- board text added: "VCC"

Commit message: Prepare for v0.3.0
Parts:
- added ?: , , F.Cu at (178.5, 113.5)
- added ?: , , F.Cu at (178.5, 116.5)
Routing:
- net unconnected-(U1-BAT-Pad12): track 0.00 -> 21.3 mm
- net Net-(BZ1--): track 70.5 -> 76.2 mm
- net Net-(U1-SDA): track 75.5 -> 77.0 mm
- added copper zone on B.Cu, net Net-(BZ1--)
- added copper zone on F.Cu, net Net-(BZ1--)
Other:
- board text added: "B+"
- board text added: "B-"

Commit message: Upload v0.3.7 contents
Parts:
- added D2 (x2): SM4007, Diode_SMD:D_MELF, B.Cu at (139.0, 113.0)
- added Q1: BC547, Package_TO_SOT_THT:TO-92_Inline, F.Cu at (131.5, 118.0)
- added R2: R, Resistor_THT:R_Axial_DIN0204_L3.6mm_D1.6mm_P5.08mm_Horizontal, F.Cu at (143.5, 110.0)
- U2: value module_mpu6050 -> module_adxl345; footprint usini_sensors:module_mpu6050 -> usini_sensors:module_adxl345
- moved U2 2.56 mm to (154.5, 110.0)
- moved BZ1 1.58 mm to (135.0, 116.0)
Connections:
- ? pad B-: Net-(BZ1--) -> Net-(Q1-E)
- R1 pad 2: Net-(BZ1--) -> Net-(Q1-E)
- SW1 pad 1: Net-(BZ1--) -> Net-(Q1-E)
- SW2 pad 1: Net-(BZ1--) -> Net-(Q1-E)
- U1 pad 10: unconnected-(U1-USB-Pad10) -> Net-(BZ1-+)
- U1 pad 16: Net-(BZ1--) -> Net-(Q1-E)
- U1 pad 3: Net-(BZ1-+) -> Net-(U1-D8)
- U2 pad 1: Net-(U2-VCC) -> Net-(Q1-E)
- U2 pad 2: Net-(BZ1--) -> Net-(U2-VCC)
- U2 pad 3: Net-(U1-SCL) -> unconnected-(U2-CS-Pad3)
- U2 pad 4: Net-(U1-SDA) -> Net-(U1-A2)
- U2 pad 7: unconnected-(U2-ADD-Pad7) -> Net-(U1-SDA)
- U2 pad 8: Net-(U1-A2) -> Net-(U1-SCL)
- U3 pad 1: Net-(U2-VCC) -> Net-(Q1-E)
- U3 pad 2: Net-(BZ1--) -> Net-(U2-VCC)
- U3 pad 1: Net-(BZ1--) -> Net-(Q1-E)
Routing:
- net Net-(Q1-E): track 0.00 -> 100.5 mm
- net Net-(BZ1-+): track 12.9 -> 88.4 mm
- net Net-(BZ1--): track 76.2 -> 16.5 mm
- net Net-(U1-SDA): track 77.0 -> 52.6 mm
- net Net-(U1-D8): track 0.00 -> 23.5 mm
- net Net-(Q1-B): track 0.00 -> 21.0 mm
- net Net-(U1-SCL): track 58.1 -> 71.6 mm
- net Net-(U2-VCC): track 62.0 -> 69.9 mm
- net Net-(U1-A2): track 9.12 -> 5.26 mm
- net unconnected-(U1-BAT-Pad12): track 21.3 -> 23.9 mm
- net Net-(U1-D0): track 15.8 -> 16.4 mm
- net Net-(U1-D3): track 40.8 -> 41.4 mm
- added copper zone on B.Cu, net Net-(U1-SDA)
- removed copper zone on B.Cu, net Net-(BZ1--)
- removed copper zone on F.Cu, net Net-(BZ1--)

Commit message: Bump to v0.3.8
Routing:
- net Net-(U1-SCL): track 71.6 -> 67.9 mm
- net Net-(U1-SDA): track 52.6 -> 50.8 mm
- net Net-(U1-D3): track 41.4 -> 42.3 mm
- added copper zone on F.Cu, net Net-(Q1-E)
- removed copper zone on B.Cu, net Net-(U1-SDA)

Commit message: v0.3.8: Add pins text for BJT
Other:
- board text added: "B"
- board text added: "BC547"
- board text added: "C"
- board text added: "E"
Changed lines of the file:
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@@
 			(drillshape 0)
 			(scaleselection 1)
-			(outputdirectory "../out-v0-3-7/")
+			(outputdirectory "../out-v0-3-8/")
 		)
 	)
@@
 		)
 	)
+	(gr_text "C"
+		(at 133 119 0)
+		(layer "B.SilkS")
+		(effects
+			(font
+				(size 1 0.7)
+				(thickness 0.1)
+			)
+			(justify left bottom mirror)
+		)
+	)
 	(gr_text "SDA"
 		(at 130.5 121 0)
@@
 		(layer "B.SilkS")
 		(effects
+			(font
+				(size 1 0.7)
+				(thickness 0.1)
+			)
+			(justify left bottom mirror)
+		)
+	)
+	(gr_text "E"
+		(at 133 116 0)
+		(layer "B.SilkS")
+		(effects
+			(font
+				(size 1 0.7)
+				(thickness 0.1)
+			)
+			(justify left bottom mirror)
+		)
+	)
+	(gr_text "BC547"
+		(at 134 120.5 0)
+		(layer "B.SilkS")
+		(effects
+			(font
+				(size 1 0.7)
+				(thickness 0.1)
+			)
+			(justify left bottom mirror)
+		)
+	)
+	(gr_text "B"
+		(at 133 117.5 0)
+		(layer "B.SilkS")
+		(effects

Commit message: Version v0.3.9
Parts:
- moved BZ1 10.5 mm to (145.3, 118.0), turned to 180 degrees
- moved D2 2.06 mm to (141.0, 113.5), turned to 180 degrees (x2)
Routing:
- net Net-(BZ1-+): track 88.4 -> 64.7 mm
- net Net-(BZ1--): track 16.5 -> 12.3 mm
- net Net-(U1-SCL): track 67.9 -> 67.4 mm

Commit message: Version 0.4!
Parts:
- moved ? 0.50 mm to (179.0, 113.5)
- moved ? 0.50 mm to (179.0, 116.5)
Routing:
- net Net-(BZ1-+): track 64.7 -> 67.7 mm
- net Net-(Q1-B): track 21.0 -> 18.3 mm
Changed lines of the file:
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@@
 		(title "Sidekick PCB")
 		(date "2025-08-14")
-		(rev "0.3.9")
+		(rev "0.4.0")
 	)
 	(layers
@@
 	(footprint ""
 		(layer "F.Cu")
-		(at 178.5 113.5)
+		(at 179 113.5)
 		(property "Reference" ""
 			(at 0 0 0)
@@
 	(footprint ""
 		(layer "F.Cu")
-		(at 178.5 116.5)
+		(at 179 116.5)
 		(property "Reference" ""
 			(at 0 0 0)
@@
 	)
 	(segment
-		(start 177.5 123)
-		(end 173.5 123)
+		(start 175.5 126.5)
+		(end 175.5 123.5)
 		(width 0.5)
 		(layer "F.Cu")
@@
 	)
 	(segment
-		(start 173.5 123)
-		(end 173 123.5)
+		(start 174.693118 127.306882)
+		(end 175.5 126.5)
 		(width 0.5)
 		(layer "F.Cu")
@@
 	)
 	(segment
-		(start 172.693118 127.306882)
-		(end 164.625 127.306882)
+		(start 164.625 127.306882)
+		(end 174.693118 127.306882)
 		(width 0.5)
 		(layer "F.Cu")
@@
 	)
 	(segment
-		(start 178.5 122)
-		(end 177.5 123)
+		(start 175.5 123.5)
+		(end 176 123)
 		(width 0.5)
 		(layer "F.Cu")
@@
 	)
 	(segment
-		(start 173 123.5)
-		(end 173 127)
+		(start 178 123)
+		(end 179 122)
 		(width 0.5)
 		(layer "F.Cu")
@@
 	)
 	(segment
-		(start 173 127)
-		(end 172.693118 127.306882)
+		(start 176 123)
+		(end 178 123)
 		(width 0.5)
 		(layer "F.Cu")
@@
 	)
 	(segment
-		(start 178.5 116.5)
-		(end 178.5 122)
+		(start 179 122)
+		(end 179 116.5)
 		(width 0.5)
 		(layer "F.Cu")
@@
 	)
 	(segment
-		(start 130 128)
-		(end 131 129)
+		(start 131 129)
+		(end 159 129)
 		(width 0.5)
 		(layer "F.Cu")
@@
 	)
 	(segment
-		(start 145.3 118)
-		(end 145.3 123.7)
-		(width 0.2)
+		(start 147 123.5)
+		(end 146.5 124)
+		(width 0.5)
 		(layer "F.Cu")
 		(net 27)
@@
 	)
 	(segment
-		(start 159.525 128.475)
-		(end 159.525 127.306882)
+		(start 136 124)
+		(end 134.5 122.5)
 		(width 0.5)
 		(layer "F.Cu")
@@
 	)
 	(segment
-		(start 145 124)
-		(end 136 124)
-		(width 0.2)
+		(start 130 128)
+		(end 131 129)
+		(width 0.5)
 		(layer "F.Cu")
 		(net 27)
 	)
 	(segment
-		(start 131 129)
-		(end 159 129)
+		(start 159.525 128.475)
+		(end 159.525 127.306882)
 		(width 0.5)
 		(layer "F.Cu")
@@
 	)
 	(segment
-		(start 136 124)
-		(end 134.5 122.5)
-		(width 0.2)
+		(start 146.5 124)
+		(end 136 124)
+		(width 0.5)
 		(layer "F.Cu")
 		(net 27)
 	)
 	(segment
-		(start 130.5 122.5)
-		(end 130 123)
+		(start 147 118.5)
+		(end 147 123.5)
 		(width 0.5)
 		(layer "F.Cu")
@@
 		(start 134.5 122.5)
 		(end 130.5 122.5)
-		(width 0.2)
+		(width 0.5)
 		(layer "F.Cu")
 		(net 27)
 	)
 	(segment
-		(start 130 123)
-		(end 130 128)
+		(start 145.3 118)
+		(end 146.5 118)
+		(width 0.5)
+		(layer "F.Cu")
+		(net 27)
+	)
+	(segment
+		(start 146.5 118)
+		(end 147 118.5)
 		(width 0.5)
 		(layer "F.Cu")
@@
 	)
 	(segment
-		(start 145.3 123.7)
-		(end 145 124)
-		(width 0.2)
+		(start 130 123)
+		(end 130 128)
+		(width 0.5)
+		(layer "F.Cu")
+		(net 27)
+	)
+	(segment
+		(start 130.5 122.5)
+		(end 130 123)
+		(width 0.5)
 		(layer "F.Cu")
 		(net 27)
@@
 	)
 	(segment
+		(start 179 112)
+		(end 179 113.5)
+		(width 0.5)
+		(layer "F.Cu")
+		(net 31)
+	)
+	(segment
 		(start 170 112)
 		(end 174.19 112)
@@
 	)
 	(segment
-		(start 175 111.19)
-		(end 178.19 111.19)
+		(start 169 113)
+		(end 170 112)
 		(width 0.5)
 		(layer "F.Cu")
@@
 	)
 	(segment
-		(start 169 113)
-		(end 170 112)
+		(start 178.19 111.19)
+		(end 179 112)
 		(width 0.5)
 		(layer "F.Cu")
@@
 	)
 	(segment
-		(start 178.19 111.19)
-		(end 178.5 111.5)
+		(start 175 111.19)
+		(end 178.19 111.19)
 		(width 0.5)
 		(layer "F.Cu")
@@
 	)
 	(segment
-		(start 178.5 111.5)
-		(end 178.5 113.5)
-		(width 0.5)
-		(layer "F.Cu")
-		(net 31)
-	)
-	(segment
 		(start 169.625 109.783882)
 		(end 169.763 109.921882)
@@
 	)
 	(segment
-		(start 130 112)
-		(end 130.5 111.5)
-		(width 0.2)
-		(layer "F.Cu")
-		(net 32)
-	)
-	(segment
-		(start 143.5 111)
-		(end 143.5 110)
-		(width 0.2)
-		(layer "F.Cu")
-		(net 32)
-	)
-	(segment
-		(start 131.5 116.729999)
-		(end 130.229999 116.729999)
+		(start 135.5 110.5)
+		(end 135.5 116.5)
 		(width 0.2)
 		(layer "F.Cu")
@@
 	)
 	(segment
-		(start 130 116.5)
-		(end 130 112)
+		(start 143.5 110)
+		(end 136 110)
 		(width 0.2)
 		(layer "F.Cu")
@@
 	)
 	(segment
-		(start 130.229999 116.729999)
-		(end 130 116.5)
+		(start 136 110)
+		(end 135.5 110.5)
 		(width 0.2)
 		(layer "F.Cu")
@@
 	)
 	(segment
-		(start 143 111.5)
-		(end 143.5 111)
+		(start 135.270001 116.729999)
+		(end 131.5 116.729999)
 		(width 0.2)
 		(layer "F.Cu")
@@
 	)
 	(segment
-		(start 130.5 111.5)
-		(end 143 111.5)
+		(start 135.5 116.5)
+		(end 135.270001 116.729999)
 		(width 0.2)
 		(layer "F.Cu")
@@
 		(min_thickness 0.25)
 		(filled_areas_thickness no)
-		(fill yes
+		(fill
 			(thermal_gap 0.5)
 			(thermal_bridge_width 0.5)
@@
 		(polygon
 			(pts
-				(xy 151.5 116.5) (xy 151.5 119.5) (xy 170.5 119.5) (xy 170.5 113.5) (xy 177 113.5) (xy 177 114.5)
-				(xy 180 114.5) (xy 180 110.5) (xy 171 110.5) (xy 170.5 111) (xy 168.5 112) (xy 168.5 116.5)
+				(xy 151.5 116.5) (xy 151.5 119.5) (xy 170.5 119.5) (xy 170.5 113.5) (xy 177 113.5) (xy 177 115)
+				(xy 180.5 115) (xy 180.5 110.5) (xy 171 110.5) (xy 170.5 111) (xy 168.5 112) (xy 168.5 116.5)
 			)
 		)

Commit message: Revision v0.4.2
Routing:
- net Net-(U2-VCC): track 69.9 -> 66.7 mm
Other:
- board text added: "C3"
- board text added: "GLYPH"
- board text added: "Hack me for a digital cookie!"
- board text added: "MADE FOR"
- board text added: "Sidekick PCB v0"
