File: sidekick.kicad_pcb (KiCad board)
At the start: 2 copper layers, 64.5 x 26.5 mm, 15 parts, among them Q1 BC547, SW1 SW_PUSH_6mm_H5mm, SW2 SW_PUSH_6mm_H5mm, U2 module_adxl345, U3 DM-OLED096-636

Commit message: Bump to v0.4.8
Parts:
- removed the D2 at (141.0, 113.5)
- SW1, SW2: moved to B.Cu
- moved SW1 6.50 mm to (169.2, 118.2), turned to 180 degrees
- moved SW2 6.50 mm to (159.2, 118.2), turned to 180 degrees
- moved ? 1.12 mm to (174.0, 121.5)
Connections:
- U1 pad 10: Net-(BZ1-+) -> unconnected-(U1-USB-Pad10)
- U1 pad 15: Net-(U2-VCC) -> Net-(BZ1-+)
- U2 pad 2: Net-(U2-VCC) -> Net-(BZ1-+)
- U3 pad 2: Net-(U2-VCC) -> Net-(BZ1-+) (x2)
Routing:
- net Net-(U2-VCC): track 66.7 -> 0.00 mm
- net Net-(BZ1-+): track 67.7 -> 95.4 mm
- net Net-(U1-D3): track 42.3 -> 43.5 mm
- net Net-(Q1-E): track 100.5 -> 101.6 mm
Other:
- board text added: "Hack me for a"
- board text added: "digital cookie!"
- board text removed: "Hack me for a digital cookie!"
