File: sidekick.kicad_pcb (KiCad board)
At the start: 2 copper layers, 64.5 x 26.5 mm, 14 parts, among them Q1 BC547, SW1 SW_PUSH_6mm_H5mm, SW2 SW_PUSH_6mm_H5mm, U2 module_adxl345, U3 DM-OLED096-636

Commit message: Update to v0.5.0
Routing:
- net Net-(U1-D3): track 43.2 -> 35.8 mm
- net Net-(Q1-E): track 101.6 -> 102.4 mm

Commit message: Bump to 0.5.1
Routing:
- net Net-(BZ1-+): track 95.4 -> 94.5 mm
Changed lines of the file:
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@@
 		(title "Sidekick PCB")
 		(date "2025-08-14")
-		(rev "0.5.0")
+		(rev "0.5.1")
 	)
 	(layers
@@
 			(drillshape 0)
 			(scaleselection 1)
-			(outputdirectory "../out-v0-5-0/")
+			(outputdirectory "../out-v0-5-1/")
 		)
 	)
@@
 	)
 	(segment
-		(start 169.5 106.781882)
-		(end 169.625 106.906882)
-		(width 0.5)
-		(layer "F.Cu")
-		(net 26)
-	)
-	(segment
-		(start 169 105)
-		(end 130 105)
-		(width 0.5)
-		(layer "F.Cu")
-		(net 26)
-	)
-	(segment
 		(start 125.5 112.5)
 		(end 125.5 113.5)
@@
 	)
 	(segment
-		(start 169 105)
-		(end 169.5 105.5)
+		(start 128.77 115.73)
+		(end 127.5 115.73)
 		(width 0.5)
 		(layer "F.Cu")
@@
 	)
 	(segment
-		(start 128.77 115.73)
-		(end 127.5 115.73)
+		(start 126 109)
+		(end 125.5 109.5)
 		(width 0.5)
 		(layer "F.Cu")
@@
 	)
 	(segment
-		(start 128.5 109)
-		(end 126 109)
-		(width 0.5)
-		(layer "F.Cu")
-		(net 26)
-	)
-	(segment
 		(start 127.5 115.5)
 		(end 127.5 115.54)
@@
 	(segment
 		(start 169.5 105.5)
-		(end 169.5 106.781882)
+		(end 169 105)
 		(width 0.5)
 		(layer "F.Cu")
@@
 	)
 	(segment
-		(start 129.5 105.5)
-		(end 129.5 108)
-		(width 0.5)
-		(layer "F.Cu")
-		(net 26)
-	)
-	(segment
-		(start 125.5 109.5)
-		(end 125.5 112.5)
-		(width 0.5)
-		(layer "F.Cu")
-		(net 26)
-	)
-	(segment
 		(start 125.19 113.19)
 		(end 124.75 113.19)
@@
 	)
 	(segment
-		(start 130 105)
-		(end 129.5 105.5)
-		(width 0.5)
-		(layer "F.Cu")
-		(net 26)
-	)
-	(segment
 		(start 128.77 115.77)
 		(end 129.5 116.5)
@@
 	)
 	(segment
+		(start 169 105)
+		(end 131.5 105)
+		(width 0.5)
+		(layer "F.Cu")
+		(net 26)
+	)
+	(segment
 		(start 145.3 118)
 		(end 143.3 120)
@@
 	)
 	(segment
-		(start 126 109)
-		(end 125.5 109.5)
+		(start 129.5 107)
+		(end 129.5 108)
 		(width 0.5)
 		(layer "F.Cu")
@@
 	)
 	(segment
+		(start 169.625 106.906882)
+		(end 169.5 106.781882)
+		(width 0.5)
+		(layer "F.Cu")
+		(net 26)
+	)
+	(segment
+		(start 131.5 105)
+		(end 129.5 107)
+		(width 0.5)
+		(layer "F.Cu")
+		(net 26)
+	)
+	(segment
+		(start 125.5 109.5)
+		(end 125.5 112.5)
+		(width 0.5)
+		(layer "F.Cu")
+		(net 26)
+	)
+	(segment
+		(start 169.5 106.781882)
+		(end 169.5 105.5)
+		(width 0.5)
+		(layer "F.Cu")
+		(net 26)
+	)
+	(segment
+		(start 128.5 109)
+		(end 126 109)
+		(width 0.5)
+		(layer "F.Cu")
+		(net 26)
+	)
+	(segment
 		(start 125.44 112.5)
 		(end 124.75 113.19)
@@
 	)
 	(zone
-		(net 30)
-		(net_name "Net-(Q1-E)")
-		(layer "F.Cu")
-		(hatch edge 0.5)
-		(connect_pads
-			(clearance 0.5)
-		)
-		(min_thickness 0.25)
-		(filled_areas_thickness no)
-		(fill yes
-			(thermal_gap 0.5)
-			(thermal_bridge_width 0.5)
-		)
-		(polygon
-			(pts
-				(xy 156 111.5) (xy 155.5 112) (xy 155.5 114) (xy 155 115) (xy 150.5 115) (xy 150.5 119.25) (xy 151 120)
-				(xy 170.5 120) (xy 171.5 119) (xy 171.5 116.5) (xy 171.5 115) (xy 172 114) (xy 178.5 114) (xy 178.5 114)
-				(xy 179.5 114) (xy 180 112.125) (xy 178.839431 110.5) (xy 171.428634 110.5) (xy 170.5 109.5) (xy 169 109.5)
-				(xy 169 111) (xy 168.5 111.5)
-			)
-		)
-	)
-	(zone
 		(net 19)
 		(net_name "Net-(U1-SDA)")
@@
 	)
 	(zone
-		(net 19)
-		(net_name "Net-(U1-SDA)")
+		(net 30)
+		(net_name "Net-(Q1-E)")
 		(layer "F.Cu")
-		(name "$teardrop_padvia$")
-		(hatch none 0.1)
-		(priority 30000)
-		(attr
-			(teardrop
-				(type padvia)
-			)
-		)
-		(connect_pads yes
-			(clearance 0)
+		(hatch edge 0.5)
+		(connect_pads
+			(clearance 0.5)
 		)
-		(min_thickness 0.0254)
+		(min_thickness 0.25)
 		(filled_areas_thickness no)
 		(fill yes
 			(thermal_gap 0.5)
 			(thermal_bridge_width 0.5)
-			(island_removal_mode 1)
-			(island_area_min 10)
 		)
 		(polygon
 			(pts
-				(xy 124.493512 120.91) (xy 124.493512 120.71) (xy 123.4189 120.183072) (xy 122.999 120.81) (xy 123.4189 121.436928)
+				(xy 156 111.5) (xy 155.5 112) (xy 155.5 114) (xy 155 115) (xy 150.5 115) (xy 150.5 119.25) (xy 151 120)
+				(xy 170.5 120) (xy 171.5 119) (xy 171.5 116.5) (xy 171.5 115) (xy 172 114) (xy 178.5 114) (xy 179.5 114)
+				(xy 180 112.125) (xy 178.839431 110.5) (xy 171.428634 110.5) (xy 170.5 109.5) (xy 169 109.5) (xy 169 111)
+				(xy 168.5 111.5)
 			)
 		)
 	)
 	(zone
-		(net 23)
-		(net_name "Net-(U1-SCL)")
+		(net 19)
+		(net_name "Net-(U1-SDA)")
 		(layer "F.Cu")
 		(name "$teardrop_padvia$")
 		(hatch none 0.1)
-		(priority 30002)
+		(priority 30000)
 		(attr
 			(teardrop
@@
 		(polygon
 			(pts
-				(xy 126.006488 118.17) (xy 126.006488 118.37) (xy 127.0811 118.896928) (xy 127.501 118.27) (xy 127.0811 117.643072)
+				(xy 124.493512 120.91) (xy 124.493512 120.71) (xy 123.4189 120.183072) (xy 122.999 120.81) (xy 123.4189 121.436928)
 			)
 		)
@@
 		(polygon
 			(pts
-				(xy 124.493512 118.37) (xy 124.493512 118.17) (xy 123.4189 117.643072) (xy 122.999 118.27) (xy 123.4189 118.896928)
+				(xy 126.006488 118.17) (xy 126.006488 118.37) (xy 127.0811 118.896928) (xy 127.501 118.27) (xy 127.0811 117.643072)
 			)
 		)
 	)
 	(zone
-		(net 19)
-		(net_name "Net-(U1-SDA)")
-		(layer "B.Cu")
+		(net 23)
+		(net_name "Net-(U1-SCL)")
+		(layer "F.Cu")
 		(name "$teardrop_padvia$")
 		(hatch none 0.1)
-		(priority 30001)
+		(priority 30002)
 		(attr
 			(teardrop
@@
 		(polygon
 			(pts
-				(xy 138.750904 125.609483) (xy 138.609483 125.750904) (xy 138.391333 127.041055) (xy 139.225707 127.207589)
-				(xy 139.697235 126.500133)
+				(xy 124.493512 118.37) (xy 124.493512 118.17) (xy 123.4189 117.643072) (xy 122.999 118.27) (xy 123.4189 118.896928)
 			)
 		)
@@
 		(name "$teardrop_padvia$")
 		(hatch none 0.1)
-		(priority 30003)
+		(priority 30002)
 		(attr
 			(teardrop
@@
 		(polygon
 			(pts
-				(xy 154.4 111.509358) (xy 154.6 111.509358) (xy 155.17358 110.423345) (xy 154.54 109.999) (xy 153.90642 110.423345)
+				(xy 128.580361 121.841783) (xy 128.721783 121.700361) (xy 128.126928 120.3911) (xy 127.499293 120.809293)
+				(xy 127.352902 121.549512)
 			)
 		)
@@
 	)
 	(zone
-		(net 23)
-		(net_name "Net-(U1-SCL)")
+		(net 19)
+		(net_name "Net-(U1-SDA)")
 		(layer "B.Cu")
 		(name "$teardrop_padvia$")
 		(hatch none 0.1)
-		(priority 30004)
+		(priority 30003)
 		(attr
 			(teardrop
@@
 		(polygon
 			(pts
-				(xy 151.9 111.509358) (xy 152.1 111.509358) (xy 152.63358 110.423345) (xy 152 109.999) (xy 151.36642 110.423345)
+				(xy 154.4 111.509358) (xy 154.6 111.509358) (xy 155.17358 110.423345) (xy 154.54 109.999) (xy 153.90642 110.423345)
 			)
 		)
@@
 		(name "$teardrop_padvia$")
 		(hatch none 0.1)
-		(priority 30000)
+		(priority 30006)
 		(attr
 			(teardrop
@@
 		(polygon
 			(pts
-				(xy 135.359403 127.999176) (xy 135.500824 128.140597) (xy 136.990827 128.040549) (xy 136.825707 127.206175)
-				(xy 136.118251 126.734647)
+				(xy 128.485361 119.396783) (xy 128.626783 119.255361) (xy 128.239512 118.122902) (xy 127.499293 118.269293)
+				(xy 127.352902 119.009512)
 			)
 		)
 	)
 	(zone
-		(net 19)
-		(net_name "Net-(U1-SDA)")
+		(net 23)
+		(net_name "Net-(U1-SCL)")
 		(layer "B.Cu")
 		(name "$teardrop_padvia$")
 		(hatch none 0.1)
-		(priority 30002)
+		(priority 30005)
 		(attr
 			(teardrop
@@
 		(polygon
 			(pts
-				(xy 128.580361 121.841783) (xy 128.721783 121.700361) (xy 128.126928 120.3911) (xy 127.499293 120.809293)
-				(xy 127.352902 121.549512)
+				(xy 124.493512 118.37) (xy 124.493512 118.17) (xy 123.4189 117.643072) (xy 122.999 118.27) (xy 123.4189 118.896928)
 			)
 		)
@@
 		(name "$teardrop_padvia$")
 		(hatch none 0.1)
-		(priority 30005)
+		(priority 30004)
 		(attr
 			(teardrop
@@
 		(polygon
 			(pts
-				(xy 124.493512 118.37) (xy 124.493512 118.17) (xy 123.4189 117.643072) (xy 122.999 118.27) (xy 123.4189 118.896928)
+				(xy 151.9 111.509358) (xy 152.1 111.509358) (xy 152.63358 110.423345) (xy 152 109.999) (xy 151.36642 110.423345)
+			)
+		)
+	)
+	(zone
+		(net 19)
+		(net_name "Net-(U1-SDA)")
+		(layer "B.Cu")
+		(name "$teardrop_padvia$")
+		(hatch none 0.1)
+		(priority 30001)
+		(attr
+			(teardrop
+				(type padvia)
+			)
+		)
+		(connect_pads yes
+			(clearance 0)
+		)
+		(min_thickness 0.0254)
+		(filled_areas_thickness no)
+		(fill yes
+			(thermal_gap 0.5)
+			(thermal_bridge_width 0.5)
+			(island_removal_mode 1)
+			(island_area_min 10)
+		)
+		(polygon
+			(pts
+				(xy 138.750904 125.609483) (xy 138.609483 125.750904) (xy 138.391333 127.041055) (xy 139.225707 127.207589)
+				(xy 139.697235 126.500133)
 			)
 		)
@@
 		(name "$teardrop_padvia$")
 		(hatch none 0.1)
-		(priority 30006)
+		(priority 30000)
 		(attr
 			(teardrop
@@
 		(polygon
 			(pts
-				(xy 128.485361 119.396783) (xy 128.626783 119.255361) (xy 128.239512 118.122902) (xy 127.499293 118.269293)
-				(xy 127.352902 119.009512)
+				(xy 135.359403 127.999176) (xy 135.500824 128.140597) (xy 136.990827 128.040549) (xy 136.825707 127.206175)
+				(xy 136.118251 126.734647)
 			)
 		)
