File: sidekick.kicad_sch (KiCad schematic)
At the start: 0 parts

Commit message: Add schematic and placeholder pcb
Parts:
- added BZ1: Buzzer, Buzzer_Beeper:Buzzer_12x9.5RM7.6, symbol Device:Buzzer
- added R1: R, Resistor_THT:R_Axial_DIN0207_L6.3mm_D2.5mm_P7.62mm_Horizontal, symbol Device:R
- added SW1, SW2: SW_PUSH_6mm_H5mm, Button_Switch_THT:SW_PUSH_6mm_H5mm, symbol Switch:SW_DIP_x01
- added U1: ~, PCBCUPID-GLYPHC3-Footprint:GlyphC3, symbol GlyphC3:GLYPHC3
- added U2: module_mpu6050, usini_sensors:module_mpu6050, symbol usini_sensors:module_mpu6050
- added U3: DM-OLED096-636, DM-OLED096-636:MODULE_DM-OLED096-636, symbol DM-OLED096-636:DM-OLED096-636
Connections:
- new net: U1.1 (SCL), U2.3 (SCL), U3.3 (SCL)
- new net: U1.15 (3V3), U2.1 (VCC), U3.2 (VCC_IN)
- new net: BZ1.2 (-), R1.2, SW1.1, SW2.1, U1.16 (GND), U2.2 (GND), U3.1 (GND)
- new net: U1.19 (A2), U2.8 (INT)
- new net: U1.2 (SDA), U2.4 (SDA), U3.4 (SDA)
- new net: BZ1.1 (+), U1.3 (D8)
- new net: R1.1, U1.6 (D3)
- new net: SW1.2, U1.8 (D1)
- new net: SW2.2, U1.9 (D0)

Commit message: Update to v0.2.5
Connections:
- net at U1.8 (D1): now also SW2.2; no longer SW1.2
- net at U1.9 (D0): now also SW1.2; no longer SW2.2
Other:
- title: (none) -> Sidekick PCB
- moved on the sheet: BZ1, R1, SW1, SW2, U1, U2, U3

Commit message: Upload v0.3.7 contents
Parts:
- removed U2: module_mpu6050, usini_sensors:module_mpu6050, symbol usini_sensors:module_mpu6050
- added D2: SM4007, Diode_SMD:D_MELF, symbol Diode:SM4007
- added Q1: BC547, Package_TO_SOT_THT:TO-92_Inline, symbol Transistor_BJT:BC547
- added R2: R, Resistor_THT:R_Axial_DIN0204_L3.6mm_D1.6mm_P5.08mm_Horizontal, symbol Device:R
- added U2: module_adxl345, usini_sensors:module_adxl345, symbol usini_sensors:module_adxl345
Connections:
- net at U1.1 (SCL), U3.3 (SCL): now also U2.8 (SCL)
- net at U1.10 (USB): now also BZ1.1 (+), D2.1 (K)
- net at U1.15 (3V3), U3.2 (VCC_IN): now also U2.2 (VCC)
- net at R1.2, SW1.1, SW2.1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: now also Q1.3 (E), U2.1 (GND); no longer BZ1.2 (-)
- net at U1.19 (A2): now also U2.4 (INT1)
- net at U1.2 (SDA), U3.4 (SDA): now also U2.7 (SDA)
- net at U1.3 (D8): now also R2.2; no longer BZ1.1 (+)
- new net: BZ1.2 (-), D2.2 (A), Q1.1 (C)
- new net: Q1.2 (B), R2.1
Other:
- moved on the sheet: BZ1

Commit message: Bump to v0.4.8
Connections:
- net at BZ1.1 (+), D2.1 (K): now also U1.15 (3V3), U2.2 (VCC), U3.2 (VCC_IN); no longer U1.10 (USB)
Other:
- moved on the sheet: BZ1, D2, Q1, R1, R2, SW1, SW2, U1, U2, U3
